Commit message: MyCobot simulation complete

File: src/mycobot_ros2/mycobot_description/urdf/parts/G_base.urdf.xacro (robot description, xacro)
@@ -10,5 +10,5 @@
       <visual>
         <geometry>
-          <mesh filename="file://$(find mycobot_description)/meshes/G_base/visual/G_base.dae"/>
+          <mesh filename="package://mycobot_description/meshes/G_base/visual/G_base.dae"/>
         </geometry>
         <origin xyz = "0.0 0 -0.03" rpy = "0 0 ${pi/2}"/>
@@ -16,5 +16,5 @@
       <collision>
         <geometry>
-          <mesh filename="file://$(find mycobot_description)/meshes/G_base/visual/G_base.dae"/>
+          <mesh filename="package://mycobot_description/meshes/G_base/visual/G_base.dae"/>
         </geometry>
         <origin xyz = "0.0 0 -0.03" rpy = "0 0 ${pi/2}"/>

File: src/mycobot_ros2/mycobot_description/urdf/parts/adaptive_gripper.urdf.xacro (robot description, xacro)
@@ -29,5 +29,5 @@
       <visual>
         <geometry>
-          <mesh filename="file://$(find mycobot_description)/meshes/adaptive_gripper/visual/gripper_base.dae"/>
+          <mesh filename="package://mycobot_description/meshes/adaptive_gripper/visual/gripper_base.dae"/>
         </geometry>
         <origin xyz="0 0 -0.012" rpy="0 0 0"/>
@@ -35,5 +35,5 @@
       <collision>
         <geometry>
-          <mesh filename="file://$(find mycobot_description)/meshes/adaptive_gripper/visual/gripper_base.dae"/>
+          <mesh filename="package://mycobot_description/meshes/adaptive_gripper/visual/gripper_base.dae"/>
         </geometry>
         <origin xyz="0 0 -0.012" rpy="0 0 0"/>
@@ -45,10 +45,9 @@
       <xacro:insert_block name="origin"/>
     </joint>
-    <!-- 左手指 -->
     <link name="${prefix}gripper_left1">
       <xacro:gripper_link_inertial/>
       <visual>
         <geometry>
-          <mesh filename="file://$(find mycobot_description)/meshes/adaptive_gripper/visual/gripper_left1.dae"/>
+          <mesh filename="package://mycobot_description/meshes/adaptive_gripper/visual/gripper_left1.dae"/>
         </geometry>
         <origin xyz="0.039 -0.0133 -0.012" rpy="0 0 0"/>
@@ -56,5 +55,5 @@
       <collision>
         <geometry>
-          <mesh filename="file://$(find mycobot_description)/meshes/adaptive_gripper/visual/gripper_left1.dae"/>
+          <mesh filename="package://mycobot_description/meshes/adaptive_gripper/visual/gripper_left1.dae"/>
         </geometry>
         <origin xyz="0.039 -0.0133 -0.012" rpy="0 0 0"/>
@@ -65,5 +64,5 @@
       <visual>
         <geometry>
-          <mesh filename="file://$(find mycobot_description)/meshes/adaptive_gripper/visual/gripper_left2.dae"/>
+          <mesh filename="package://mycobot_description/meshes/adaptive_gripper/visual/gripper_left2.dae"/>
         </geometry>
         <origin xyz="0.005 -0.0195 -0.012" rpy="0 0 0"/>
@@ -71,5 +70,5 @@
       <collision>
         <geometry>
-          <mesh filename="file://$(find mycobot_description)/meshes/adaptive_gripper/visual/gripper_left2.dae"/>
+          <mesh filename="package://mycobot_description/meshes/adaptive_gripper/visual/gripper_left2.dae"/>
         </geometry>
         <origin xyz="0.005 -0.0195 -0.012" rpy="0 0 0"/>
@@ -80,5 +79,5 @@
       <visual>
         <geometry>
-          <mesh filename="file://$(find mycobot_description)/meshes/adaptive_gripper/visual/gripper_left3.dae"/>
+          <mesh filename="package://mycobot_description/meshes/adaptive_gripper/visual/gripper_left3.dae"/>
         </geometry>
         <origin xyz="0.012 0.0025 -0.012" rpy="0 0 0"/>
@@ -86,5 +85,5 @@
       <collision>
         <geometry>
-          <mesh filename="file://$(find mycobot_description)/meshes/adaptive_gripper/visual/gripper_left3.dae"/>
+          <mesh filename="package://mycobot_description/meshes/adaptive_gripper/visual/gripper_left3.dae"/>
         </geometry>
         <origin xyz="0.012 0.0025 -0.012" rpy="0 0 0"/>
@@ -96,5 +95,5 @@
       <visual>
         <geometry>
-          <mesh filename="file://$(find mycobot_description)/meshes/adaptive_gripper/visual/gripper_right1.dae"/>
+          <mesh filename="package://mycobot_description/meshes/adaptive_gripper/visual/gripper_right1.dae"/>
         </geometry>
         <origin xyz="-0.039 -0.0133 -0.012" rpy="0 0 0"/>
@@ -102,5 +101,5 @@
       <collision>
         <geometry>
-          <mesh filename="file://$(find mycobot_description)/meshes/adaptive_gripper/visual/gripper_right1.dae"/>
+          <mesh filename="package://mycobot_description/meshes/adaptive_gripper/visual/gripper_right1.dae"/>
         </geometry>
         <origin xyz="-0.039 -0.0133 -0.012" rpy="0 0 0"/>
@@ -111,5 +110,5 @@
       <visual>
         <geometry>
-          <mesh filename="file://$(find mycobot_description)/meshes/adaptive_gripper/visual/gripper_right2.dae"/>
+          <mesh filename="package://mycobot_description/meshes/adaptive_gripper/visual/gripper_right2.dae"/>
         </geometry>
         <origin xyz="-0.005 -0.0195 -0.012" rpy="0 0 0"/>
@@ -117,5 +116,5 @@
       <collision>
         <geometry>
-          <mesh filename="file://$(find mycobot_description)/meshes/adaptive_gripper/visual/gripper_right2.dae"/>
+          <mesh filename="package://mycobot_description/meshes/adaptive_gripper/visual/gripper_right2.dae"/>
         </geometry>
         <origin xyz="-0.005 -0.0195 -0.012" rpy="0 0 0"/>
@@ -126,5 +125,5 @@
       <visual>
         <geometry>
-          <mesh filename="file://$(find mycobot_description)/meshes/adaptive_gripper/visual/gripper_right3.dae"/>
+          <mesh filename="package://mycobot_description/meshes/adaptive_gripper/visual/gripper_right3.dae"/>
         </geometry>
         <origin xyz="-0.012 0.0025 -0.012" rpy="0 0 0"/>
@@ -132,5 +131,5 @@
       <collision>
         <geometry>
-          <mesh filename="file://$(find mycobot_description)/meshes/adaptive_gripper/visual/gripper_right3.dae"/>
+          <mesh filename="package://mycobot_description/meshes/adaptive_gripper/visual/gripper_right3.dae"/>
         </geometry>
         <origin xyz="-0.012 0.0025 -0.012" rpy="0 0 0"/>

File: src/mycobot_ros2/mycobot_description/urdf/parts/mycobot_280_arm.urdf.xacro (robot description, xacro)
@@ -36,5 +36,5 @@
         <geometry>
         <!--- 0.0 0 -0.04  ${pi/2} 3.14159-->
-          <mesh filename="file://$(find mycobot_description)/meshes/mycobot_280/visual/joint1.dae"/>
+          <mesh filename="package://mycobot_description/meshes/mycobot_280/visual/joint1.dae"/>
         </geometry>
         <origin xyz = "0.0 0 0 " rpy = " 0 0 ${-pi/2}"/>
@@ -43,5 +43,5 @@
         <geometry>
         <!--- 0.0 0 -0.04  ${pi/2} 3.14159-->
-          <mesh filename="file://$(find mycobot_description)/meshes/mycobot_280/visual/joint1.dae"/>
+          <mesh filename="package://mycobot_description/meshes/mycobot_280/visual/joint1.dae"/>
         </geometry>
         <origin xyz = "0.0 0 0 " rpy = " 0 0 ${-pi/2}"/>
@@ -52,5 +52,5 @@
       <visual>
         <geometry>
-          <mesh filename="file://$(find mycobot_description)/meshes/mycobot_280/visual/joint2.dae"/>
+          <mesh filename="package://mycobot_description/meshes/mycobot_280/visual/joint2.dae"/>
         </geometry>
         <origin xyz = "0.0 0 -0.06096 " rpy = " 0 0 ${-pi/2}"/>
@@ -58,5 +58,5 @@
       <collision>
         <geometry>
-          <mesh filename="file://$(find mycobot_description)/meshes/mycobot_280/visual/joint2.dae"/>
+          <mesh filename="package://mycobot_description/meshes/mycobot_280/visual/joint2.dae"/>
         </geometry>
         <origin xyz = "0.0 0 -0.06096 " rpy = " 0 0 ${-pi/2}"/>
@@ -67,5 +67,5 @@
       <visual>
         <geometry>
-          <mesh filename="file://$(find mycobot_description)/meshes/mycobot_280/visual/joint3.dae"/>
+          <mesh filename="package://mycobot_description/meshes/mycobot_280/visual/joint3.dae"/>
         </geometry>
       <origin xyz = "0.0 0 0.03256 " rpy = " 0 ${-pi/2} 0"/>
@@ -73,5 +73,5 @@
       <collision>
         <geometry>
-          <mesh filename="file://$(find mycobot_description)/meshes/mycobot_280/visual/joint3.dae"/>
+          <mesh filename="package://mycobot_description/meshes/mycobot_280/visual/joint3.dae"/>
         </geometry>
         <origin xyz = "0.0 0 0.03256 " rpy = " 0 ${-pi/2} 0"/>
@@ -83,5 +83,5 @@
         <geometry>
           <!--- 0.0 0 -0.04 -->
-          <mesh filename="file://$(find mycobot_description)/meshes/mycobot_280/visual/joint4.dae"/>
+          <mesh filename="package://mycobot_description/meshes/mycobot_280/visual/joint4.dae"/>
         </geometry>
         <origin xyz = "0.0 0 0.03056 " rpy = " 0 ${-pi/2} 0"/>
@@ -90,5 +90,5 @@
         <geometry>
           <!--- 0.0 0 -0.04 -->
-          <mesh filename="file://$(find mycobot_description)/meshes/mycobot_280/visual/joint4.dae"/>
+          <mesh filename="package://mycobot_description/meshes/mycobot_280/visual/joint4.dae"/>
         </geometry>
         <origin xyz = "0.0 0 0.03056 " rpy = " 0 ${-pi/2} 0"/>
@@ -100,5 +100,5 @@
       <geometry>
         <!--- 0.0 0 -0.04 -->
-        <mesh filename="file://$(find mycobot_description)/meshes/mycobot_280/visual/joint5.dae"/>
+        <mesh filename="package://mycobot_description/meshes/mycobot_280/visual/joint5.dae"/>
       </geometry>
       <origin xyz = "0.0 -0.0 -0.0345 " rpy = "${-pi/2} 0 0"/>
@@ -107,5 +107,5 @@
       <geometry>
         <!--- 0.0 0 -0.04 -->
-        <mesh filename="file://$(find mycobot_description)/meshes/mycobot_280/visual/joint5.dae"/>
+        <mesh filename="package://mycobot_description/meshes/mycobot_280/visual/joint5.dae"/>
       </geometry>
       <origin xyz = "0.0 -0.0 -0.0345 " rpy = "${-pi/2} 0 0"/>
@@ -117,5 +117,5 @@
         <geometry>
           <!--- 0.0 0 -0.04 -->
-          <mesh filename="file://$(find mycobot_description)/meshes/mycobot_280/visual/joint6.dae"/>
+          <mesh filename="package://mycobot_description/meshes/mycobot_280/visual/joint6.dae"/>
         </geometry>
         <origin xyz = "0 0.00 -0.038 " rpy = " 0 0 0"/>
@@ -124,5 +124,5 @@
         <geometry>
           <!--- 0.0 0 -0.04 -->
-          <mesh filename="file://$(find mycobot_description)/meshes/mycobot_280/visual/joint6.dae"/>
+          <mesh filename="package://mycobot_description/meshes/mycobot_280/visual/joint6.dae"/>
         </geometry>
         <origin xyz = "0 0.00 -0.038 " rpy = " 0 0 0"/>
@@ -134,5 +134,5 @@
         <geometry>
           <!--- 0.0 0 -0.04 -->
-          <mesh filename="file://$(find mycobot_description)/meshes/mycobot_280/visual/joint7.dae"/>
+          <mesh filename="package://mycobot_description/meshes/mycobot_280/visual/joint7.dae"/>
         </geometry>
         <origin xyz = "0.0 0 -0.012 " rpy = " 0 0 0"/>
@@ -141,5 +141,5 @@
         <geometry>
           <!--- 0.0 0 -0.04 -->
-          <mesh filename="file://$(find mycobot_description)/meshes/mycobot_280/visual/joint7.dae"/>
+          <mesh filename="package://mycobot_description/meshes/mycobot_280/visual/joint7.dae"/>
         </geometry>
         <origin xyz = "0.0 0 -0.012 " rpy = " 0 0 0"/>

File: src/mycobot_ros2/mycobot_description/urdf/robots/mycobot_280.urdf.xacro (robot description, xacro)
@@ -37,8 +37,8 @@
       </xacro:if>
   </xacro:if>
-  <!-- <xacro:include filename="//package:mycobot_description/urdf/control/gazebo_sim_ros2_control.urdf.xacro" />
+  <xacro:include filename="$(find mycobot_description)/urdf/control/gazebo_sim_ros2_control.urdf.xacro" />
   <xacro:load_gazebo_sim_ros2_control_plugin robot_name="$(arg robot_name)" use_gazebo="$(arg use_gazebo)"/>
-  <xacro:include filename="//package:mycobot_description/urdf/control/mycobot_280_ros2_control.urdf.xacro" />
+  <xacro:include filename="$(find mycobot_description)/urdf/control/mycobot_280_ros2_control.urdf.xacro" />
   <xacro:mycobot_ros2_control prefix="$(arg prefix)" flange_link="$(arg flange_link)" use_gazebo="$(arg use_gazebo)"/>
-  <xacro:include filename="//package:mycobot_description/urdf/sensors/intel_rgbd_cam_d435.urdf.xacro"/> -->
+  <!-- <xacro:include filename="$(find mycobot_description)/urdf/sensors/intel_rgbd_cam_d435.urdf.xacro"/> -->
 </robot>
