Commit message: Robot and ball spawning works

File: src/table_tennis_description/urdf/control/gazebo_sim_ros2_control.urdf.xacro (robot description, xacro)
@@ -1,5 +1,5 @@
 <?xml version="1.0"?>
 <robot xmlns:xacro="http://wiki.ros.org/xacro">
-    <xacro:macro name="load_gazebo_sim_ros2_control_plugin" params="robot_name use_gazebo">
+    <xacro:macro name="load_gazebo_sim_ros2_control_plugin" params="robot_name use_gazebo namespace:=''">
         <xacro:if value="${use_gazebo}">
             <gazebo>
@@ -7,5 +7,6 @@
                     <parameters>$(find table_tennis_gazebo)/config/controllers.yaml</parameters>
                     <ros>
-                        <namespace>${robot_name}</namespace>
+                        <namespace>${namespace}</namespace>
+                        <remapping>/robot_description:=${namespace + '/' if namespace else ''}robot_description</remapping>
                     </ros>
                 </plugin>

File: src/table_tennis_description/urdf/robots/franka_with_paddle.urdf.xacro (robot description, xacro)
@@ -27,6 +27,8 @@
   <xacro:arg name="gazebo_effort" default="false"/>
   <xacro:arg name="description_pkg" default="franka_description"/>
+  <xacro:arg name="robot_namespace" default=""/>
   <!-- Compute link prefix based on arm_prefix and robot_type -->
   <xacro:property name="prefix" value="$(arg arm_prefix)"/>
+  <xacro:property name="robot_ns" value="$(arg robot_namespace)"/>
   <xacro:property name="modified_prefix" value="${prefix + '_' if prefix else ''}"/>
   <xacro:property name="robot_type_val" value="$(arg robot_type)"/>
@@ -66,3 +68,13 @@
     <origin xyz="0.05 0 0.05" rpy="0 0.785 0"/>
   </xacro:realsense_d435>
+  <!-- ros2_control integration for Gazebo -->
+  <xacro:property name="use_ros2_control" value="$(arg ros2_control)"/>
+  <xacro:property name="use_gazebo" value="$(arg gazebo)"/>
+  <xacro:if value="${use_ros2_control and use_gazebo}">
+    <!-- Include ros2_control xacro -->
+    <xacro:include filename="$(find table_tennis_description)/urdf/control/gazebo_sim_ros2_control.urdf.xacro"/>
+    <xacro:load_gazebo_sim_ros2_control_plugin robot_name="franka_table_tennis" use_gazebo="true" namespace="${robot_ns}"/>
+    <xacro:include filename="$(find table_tennis_description)/urdf/control/franka_ros2_control.urdf.xacro"/>
+    <xacro:table_tennis_ros2_control name="franka" robot_type="fr3"/>
+  </xacro:if>
 </robot>
