Commit message: Fix TF tree and simulation time synchronization
- Added clock_bridge to bridge /clock topic from Gazebo to ROS 2
  - Fixes controller_manager 'No clock received' warnings
  - Enables proper use_sim_time synchronization

- Added manual controller spawners (joint_state_broadcaster, arm_controller)
  - gz_ros2_control <parameters> tag doesn't auto-load controllers in Gazebo Harmonic
  - Controllers now properly loaded and activated

- Updated paddle collision to use visual mesh instead of box
  - More accurate collision detection for physics simulation

- Result: Complete TF tree with all joint transforms publishing
  - Dynamic TF (/tf topic) now working correctly
  - robot_state_publisher receiving sim time and publishing transforms
  - All robot links visible in Rviz with 'Transform OK' status

File: src/table_tennis_description/urdf/end_effectors/paddle/paddle.urdf.xacro (robot description, xacro)
@@ -14,8 +14,8 @@
       </visual>
       <collision>
-        <origin xyz="0 0 0.13" rpy="0 0 0"/>
+        <origin xyz="0 0 0.13" rpy="1.5708 0 0"/>
         <geometry>
-          <!-- Simplified paddle collision as single box -->
-          <box size="0.15 0.15 0.20"/>
+          <!-- Use same mesh as visual for accurate collision -->
+          <mesh filename="package://table_tennis_description/meshes/paddle/table_tennis_racket.stl" scale="0.0023 0.0023 0.0023"/>
         </geometry>
       </collision>
